Commit message: added ackermann, reverted back to skid - working

File: install/farmbot_description/share/farmbot_description/urdf/farmbot.xacro (robot description, xacro)
@@ -6,4 +6,6 @@
 <!-- <xacro:include filename="$(find farmbot_description)/urdf/gazebo_control.xacro" />  # Diff drive Controller  -->
 <xacro:include filename="$(find farmbot_description)/urdf/gazebo_control_skid.xacro" />  <!-- Skid Steer Controller-->
+<xacro:include filename="lidar.xacro" />
+<!-- <xacro:include filename="$(find farmbot_description)/urdf/gazebo_control_acker.xacro" /> --> <!-- Ackermann Controller-->
 <link name="base_link">
   <inertial>
@@ -126,11 +128,11 @@
   </collision>
 </link>
-<joint name="Revolute 1" type="fixed">
+<joint name="Revolute 1" type="fixed"> <!-- steering joint -->
   <origin xyz="-0.0625 0.0 0.087" rpy="0 0 0"/>
   <parent link="base_link"/>
   <child link="component__1__1"/>
-  <axis xyz="0.0 0.0 -0.5"/>
+  <axis xyz="0.0 0.0 1.0"/>
 </joint>
-<joint name="Revolute 2" type="continuous">
+<joint name="Revolute 2" type="continuous"> <!-- rear right wheel -->
   <origin xyz="0.161565 0.166785 0.087" rpy="0 0 0"/>
   <parent link="base_link"/>
@@ -138,5 +140,5 @@
   <axis xyz="-0.0 1.0 0.0"/>
 </joint>
-<joint name="Revolute 3" type="continuous">
+<joint name="Revolute 3" type="continuous"> <!-- rear left wheel -->
   <origin xyz="0.161565 -0.166784 0.087" rpy="0 0 0"/>
   <parent link="base_link"/>
@@ -144,5 +146,5 @@
   <axis xyz="-0.0 1.0 -0.0"/>
 </joint>
-<joint name="Revolute 4" type="continuous">
+<joint name="Revolute 4" type="continuous"> <!-- front right wheel -->
   <origin xyz="-0.161565 0.166785 0.087" rpy="0 0 0"/>
   <parent link="base_link"/>
@@ -150,5 +152,5 @@
   <axis xyz="0.0 1.0 -0.0"/>
 </joint>
-<joint name="Revolute 5" type="continuous">
+<joint name="Revolute 5" type="continuous"> <!-- front left wheel -->
   <origin xyz="-0.161565 -0.166784 0.087" rpy="0 0 0"/>
   <parent link="base_link"/>

File: install/farmbot_description/share/farmbot_description/urdf/gazebo_control_skid.xacro (robot description, xacro)
@@ -11,9 +11,9 @@
             <num_wheel_pairs>2</num_wheel_pairs>
             <!-- wheels0 -->
+            <left_joint>Revolute 5</left_joint>
+            <right_joint>Revolute 4</right_joint>
+            <!-- wheels1-->
             <left_joint>Revolute 3</left_joint>
             <right_joint>Revolute 2</right_joint>
-            <!-- wheels1-->
-            <left_joint>Revolute 5</left_joint>
-            <right_joint>Revolute 4</right_joint>
             <!-- kinematics -->
             <wheel_separation>0.23</wheel_separation>

File: install/farmbot_description/share/farmbot_description/urdf/materials.xacro (robot description, xacro)
@@ -4,3 +4,6 @@
   <color rgba="0.700 0.700 0.700 1.000"/>
 </material>
+<material name="red">
+  <color rgba="1 0 0 1"/>
+</material>
 </robot>

Commit message: Semi-working steering, check wheel links next

File: install/farmbot_description/share/farmbot_description/urdf/farmbot.xacro (robot description, xacro)
@@ -6,4 +6,5 @@
 <!-- <xacro:include filename="$(find farmbot_description)/urdf/gazebo_control.xacro" />  # Diff drive Controller  -->
 <xacro:include filename="$(find farmbot_description)/urdf/gazebo_control_skid.xacro" />  <!-- Skid Steer Controller-->
+<xacro:include filename="$(find farmbot_description)/urdf/gazebo_control_tricycle.xacro" />  <!-- trycicle Steer Controller-->
 <xacro:include filename="lidar.xacro" />
 <!-- <xacro:include filename="$(find farmbot_description)/urdf/gazebo_control_acker.xacro" /> --> <!-- Ackermann Controller-->
@@ -128,5 +129,5 @@
   </collision>
 </link>
-<joint name="Revolute 1" type="fixed"> <!-- steering joint -->
+<joint name="Revolute 1" type="continuous"> <!-- steering joint -->
   <origin xyz="-0.0625 0.0 0.087" rpy="0 0 0"/>
   <parent link="base_link"/>
@@ -147,12 +148,12 @@
 </joint>
 <joint name="Revolute 4" type="continuous"> <!-- front right wheel -->
-  <origin xyz="-0.161565 0.166785 0.087" rpy="0 0 0"/>
-  <parent link="base_link"/>
+  <origin xyz="-0.161565 0.166785 0.0" rpy="0 0 0"/>
+  <parent link="component__1__1"/>
   <child link="component__2__3"/>
   <axis xyz="0.0 1.0 -0.0"/>
 </joint>
 <joint name="Revolute 5" type="continuous"> <!-- front left wheel -->
-  <origin xyz="-0.161565 -0.166784 0.087" rpy="0 0 0"/>
-  <parent link="base_link"/>
+  <origin xyz="-0.161565 -0.166784 0.0" rpy="0 0 0"/>
+  <parent link="component__1__1"/>
   <child link="component__2__4"/>
   <axis xyz="0.0 1.0 0.0"/>

Commit message: Working! need to find how to set angle limit

File: install/farmbot_description/share/farmbot_description/urdf/farmbot.xacro (robot description, xacro)
@@ -96,5 +96,5 @@
   </inertial>
   <visual>
-    <origin xyz="0.161565 -0.166785 0.0" rpy="${pi/2} 0 0"/>
+    <origin xyz="0.161565 -.166784 0.0" rpy="${pi/2} 0 0"/>
     <geometry>
       <mesh filename="file://$(find farmbot_description)/meshes/component__2__3.stl" scale="0.001 0.001 0.001"/>
@@ -103,5 +103,5 @@
   </visual>
   <collision>
-    <origin xyz="0.161565 -0.166785 0.0" rpy="${pi/2} 0 0"/>
+    <origin xyz="0.161565 -0.166784 0.0" rpy="${pi/2} 0 0"/>
     <geometry>
       <mesh filename="file://$(find farmbot_description)/meshes/component__2__3.stl" scale="0.001 0.001 0.001"/>
@@ -116,5 +116,5 @@
   </inertial>
   <visual>
-    <origin xyz="0.161565 0.166784 0.0" rpy="${pi/2} 0 0"/>
+    <origin xyz="0.161565 0.166785 0.0" rpy="${pi/2} 0 0"/>
     <geometry>
       <mesh filename="file://$(find farmbot_description)/meshes/component__2__4.stl" scale="0.001 0.001 0.001"/>
@@ -123,5 +123,5 @@
   </visual>
   <collision>
-    <origin xyz="0.161565 0.166784 0.0" rpy="${pi/2} 0 0"/>
+    <origin xyz="0.161565 0.166785 0.0" rpy="${pi/2} 0 0"/>
     <geometry>
       <mesh filename="file://$(find farmbot_description)/meshes/component__2__4.stl" scale="0.001 0.001 0.001"/>
@@ -148,5 +148,5 @@
 </joint>
 <joint name="Revolute 4" type="continuous"> <!-- front right wheel -->
-  <origin xyz="-0.161565 0.166785 0.0" rpy="0 0 0"/>
+  <origin xyz="-0.100493 0.166785 0" rpy="0 0 0"/>
   <parent link="component__1__1"/>
   <child link="component__2__3"/>
@@ -154,5 +154,5 @@
 </joint>
 <joint name="Revolute 5" type="continuous"> <!-- front left wheel -->
-  <origin xyz="-0.161565 -0.166784 0.0" rpy="0 0 0"/>
+  <origin xyz="-0.100493 -0.166785 0" rpy="0 0 0"/>
   <parent link="component__1__1"/>
   <child link="component__2__4"/>

File: install/farmbot_description/share/farmbot_description/urdf/gazebo_control_tricycle.xacro (robot description, xacro)
@@ -10,11 +10,12 @@
             <!-- wheels -->
             <steering_joint>Revolute 1</steering_joint>
-            <actuated_wheel_joint>Revolute 2</actuated_wheel_joint>
+            <actuated_wheel_joint>Revolute 1</actuated_wheel_joint>
             <encoder_wheel_left_joint>Revolute 3</encoder_wheel_left_joint>
             <encoder_wheel_right_joint>Revolute 2</encoder_wheel_right_joint>
             <!-- kinematics -->
-            <wheel_separation>1.0</wheel_separation>
-            <encoder_wheel_diameter>0.3</encoder_wheel_diameter>
-            <actuated_wheel_diameter>0.3</actuated_wheel_diameter>
+            <wheel_separation>.23</wheel_separation>
+            <encoder_wheel_diameter>0.17</encoder_wheel_diameter>
+            <actuated_wheel_diameter>0.17</actuated_wheel_diameter>
+            <steering_angle_tolerance>.047</steering_angle_tolerance>
             <!-- limits -->
             <max_wheel_torque>20</max_wheel_torque>

File: src/farmbot_description/urdf/gazebo_control_tricycle.xacro (robot description, xacro)
@@ -10,11 +10,12 @@
             <!-- wheels -->
             <steering_joint>Revolute 1</steering_joint>
-            <actuated_wheel_joint>Revolute 2</actuated_wheel_joint>
+            <actuated_wheel_joint>Revolute 1</actuated_wheel_joint>
             <encoder_wheel_left_joint>Revolute 3</encoder_wheel_left_joint>
             <encoder_wheel_right_joint>Revolute 2</encoder_wheel_right_joint>
             <!-- kinematics -->
-            <wheel_separation>1.0</wheel_separation>
-            <encoder_wheel_diameter>0.3</encoder_wheel_diameter>
-            <actuated_wheel_diameter>0.3</actuated_wheel_diameter>
+            <wheel_separation>.23</wheel_separation>
+            <encoder_wheel_diameter>0.17</encoder_wheel_diameter>
+            <actuated_wheel_diameter>0.17</actuated_wheel_diameter>
+            <!-- <steering_angle_tolerance>.047</steering_angle_tolerance> -->
             <!-- limits -->
             <max_wheel_torque>20</max_wheel_torque>

Commit message: Able to steer, but will not drive

File: install/farmbot_description/share/farmbot_description/urdf/farmbot.xacro (robot description, xacro)
@@ -5,8 +5,8 @@
 <xacro:include filename="$(find farmbot_description)/urdf/farmbot.gazebo" />
 <!-- <xacro:include filename="$(find farmbot_description)/urdf/gazebo_control.xacro" />  # Diff drive Controller  -->
-<xacro:include filename="$(find farmbot_description)/urdf/gazebo_control_skid.xacro" />  <!-- Skid Steer Controller-->
-<xacro:include filename="$(find farmbot_description)/urdf/gazebo_control_tricycle.xacro" />  <!-- trycicle Steer Controller-->
+<!-- <xacro:include filename="$(find farmbot_description)/urdf/gazebo_control_skid.xacro" /> --> <!-- Skid Steer Controller-->
+<!-- <xacro:include filename="$(find farmbot_description)/urdf/gazebo_control_tricycle.xacro" /> --> <!-- trycicle Steer Controller-->
 <xacro:include filename="lidar.xacro" />
-<!-- <xacro:include filename="$(find farmbot_description)/urdf/gazebo_control_acker.xacro" /> --> <!-- Ackermann Controller-->
+<xacro:include filename="$(find farmbot_description)/urdf/gazebo_control_acker.xacro" /> <!-- Ackermann Controller-->
 <link name="base_link">
   <inertial>
@@ -126,4 +126,42 @@
     <geometry>
       <mesh filename="file://$(find farmbot_description)/meshes/component__2__4.stl" scale="0.001 0.001 0.001"/>
+    </geometry>
+  </collision>
+</link>
+<link name="right_steering_link">
+  <inertial>
+    <origin xyz="3.7769361843631444e-07 -3.5857001496231076e-07 -0.005961668903388867" rpy="0 0 0"/>
+    <mass value="0.01"/>
+    <inertia ixx="0.063249" iyy="0.063249" izz="0.081111" ixy="-0.0" iyz="0.0" ixz="-0.0"/>
+  </inertial>
+  <visual>
+    <origin xyz="0.0625 0.0 0.0" rpy="${pi/2} 0 0"/>
+    <geometry>
+            <box size="0.01 0.01 0.01"/>
+    </geometry>
+  </visual>
+  <collision>
+    <origin xyz="0.0625 0.0 0.0" rpy="${pi/2} 0 0"/>
+    <geometry>
+            <box size="0.01 0.01 0.01"/>
+    </geometry>
+  </collision>
+</link>
+<link name="left_steering_link">
+  <inertial>
+    <origin xyz="3.7769361843631444e-07 -3.5857001489125644e-07 0.005961691828770765" rpy="0 0 0"/>
+    <mass value="0.01"/>
+    <inertia ixx="0.063249" iyy="0.063249" izz="0.081111" ixy="0.0" iyz="0.0" ixz="0.0"/>
+  </inertial>
+  <visual>
+    <origin xyz="0.0625 0.0 0.0" rpy="${pi/2} 0 0"/>
+    <geometry>
+            <box size="0.01 0.01 0.01"/>
+    </geometry>
+  </visual>
+  <collision>
+    <origin xyz="0.0625 0.0 0.0" rpy="${pi/2} 0 0"/>
+    <geometry>
+            <box size="0.01 0.01 0.01"/>
     </geometry>
   </collision>
@@ -153,4 +191,10 @@
   <axis xyz="0.0 1.0 -0.0"/>
 </joint>
+<joint name="Revolute 6" type="continuous"> <!-- front right steering -->
+  <origin xyz="0.0625 0.0 0.0" rpy="0 0 0"/>
+  <parent link="base_link"/>
+  <child link="right_steering_link"/>
+  <axis xyz="0.0 0.0 1.0"/>
+</joint>
 <joint name="Revolute 5" type="continuous"> <!-- front left wheel -->
   <origin xyz="-0.100493 -0.166785 0" rpy="0 0 0"/>
@@ -159,3 +203,9 @@
   <axis xyz="0.0 1.0 0.0"/>
 </joint>
+<joint name="Revolute 7" type="continuous"> <!-- front left steering -->
+  <origin xyz="0.0625 0.0 0.0" rpy="0 0 0"/>
+  <parent link="base_link"/>
+  <child link="left_steering_link"/>
+  <axis xyz="0.0 0.0 1.0"/>
+</joint>
 </robot>
